Commit message: move obj

File: AM_RL/assets/urdf/ball.urdf (robot description, URDF)
Before this commit: robot ball, 1 links, 0 joints
Links:
- link base_link: geometry collision sphere radius=0.02; visual sphere radius=0.02

Commit message: tuning

File: AM_RL/assets/urdf/ball.urdf (robot description, URDF)
Before this commit: robot ball, 1 links, 0 joints
Links:
- link base_link: geometry collision sphere radius=0.05; visual sphere radius=0.05
